File: board-template.kicad_pcb (KiCad board)
At the start: 2 copper layers, 0 parts

Commit message: fix(pcb): repair unclosed sexp parenthesis from edge outline commit
Co-authored-by: aman-katyal <181611364+aman-katyal@users.noreply.github.com>
Other:
- board outline added: 100 x 100 mm
Changed lines of the file:
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@@
 		)
+	)
+	(gr_rect (start 0 0) (end 100 100)
+		(stroke (width 0.1) (type solid))
+		(fill none)
+		(layer "Edge.Cuts")
 	)
 	(embedded_fonts no)
