File: board-template.kicad_pcb (KiCad board)
At the start: 2 copper layers, 100 x 100 mm, 0 parts

Commit message: Revert task as it is closed by reviewer
Co-authored-by: aman-katyal <181611364+aman-katyal@users.noreply.github.com>
Other:
- board outline removed
Changed lines of the file:
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@@
 		)
 	)
-	(gr_rect (start 0 0) (end 100 100)
-		(stroke (width 0.1) (type solid))
-		(fill none)
-		(layer "Edge.Cuts")
-	)
 	(embedded_fonts no)
-	(gr_line (start 0 0) (end 100 0) (layer "Edge.Cuts") (width 0.1))
-	(gr_line (start 100 0) (end 100 100) (layer "Edge.Cuts") (width 0.1))
-	(gr_line (start 100 100) (end 0 100) (layer "Edge.Cuts") (width 0.1))
-	(gr_line (start 0 100) (end 0 0) (layer "Edge.Cuts") (width 0.1))
 )

Commit message: fix: resolve DRC error and CI pipeline failure
Co-authored-by: aman-katyal <181611364+aman-katyal@users.noreply.github.com>
Other:
- board outline added: 50 x 50 mm
Changed lines of the file:
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@@
 	)
 	(embedded_fonts no)
+  (gr_rect (start 0 0) (end 50 50) (stroke (width 0.1) (type solid)) (layer "Edge.Cuts"))
 )

Commit message: fix: prevent command injection in initialize-template workflow
Co-authored-by: aman-katyal <181611364+aman-katyal@users.noreply.github.com>
Other:
- board outline removed
Changed lines of the file:
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@@
 	)
 	(embedded_fonts no)
-  (gr_rect (start 0 0) (end 50 50) (stroke (width 0.1) (type solid)) (layer "Edge.Cuts"))
 )

Commit message: 🧪 [testing improvement] Add test for file not found in linter validator
This commit adds a test to cover the missing error path when a KiCad
symbol file is not found in the linter validator script.

It also fixes an issue in the `board-template.kicad_pcb` file where
the board outline (Edge.Cuts) was missing, causing CI failures when
KiBot tried to generate fabrication files.

Co-authored-by: aman-katyal <181611364+aman-katyal@users.noreply.github.com>
Other:
- board outline added: 100 x 100 mm
Changed lines of the file:
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@@
 	)
 	(embedded_fonts no)
+	(gr_line (start 0 0) (end 100 0) (layer "Edge.Cuts") (width 0.1))
+	(gr_line (start 100 0) (end 100 100) (layer "Edge.Cuts") (width 0.1))
+	(gr_line (start 100 100) (end 0 100) (layer "Edge.Cuts") (width 0.1))
+	(gr_line (start 0 100) (end 0 0) (layer "Edge.Cuts") (width 0.1))
 )
