File: board-template.kicad_pcb (KiCad board)
At the start: 2 copper layers, 0 parts

Commit message: fix(template): add edge cuts outline to PCB to unblock CI BOM generation
The KiBot interactive HTML BOM generation requires a valid board outline on the Edge.Cuts layer. This commit adds a default 100x100mm rectangular board outline to `board-template.kicad_pcb` to prevent `Failed to create BoM, error 3` errors during the GitHub Actions CI pipeline.

Co-authored-by: aman-katyal <181611364+aman-katyal@users.noreply.github.com>
Other:
- board outline added: 100 x 100 mm
Changed lines of the file:
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@@
 	)
 	(embedded_fonts no)
+	(gr_rect (start 0 0) (end 100 100) (layer "Edge.Cuts")
+		(stroke (width 0.1) (type solid))
+		(fill none)
+	)
 )
